File: PCB/usbcmacropad.kicad_sch (KiCad schematic)
At the start: 7 parts, among them SW1 SW_Push, SW2 SW_Push, SW3 SW_Push, SW4 SW_Push, U1 XIAO-RP2040-DIP

Commit message: Add files via upload
Parts:
- removed D1: SK6812MINI, LED_SMD:LED_SK6812MINI_PLCC4_3.5x3.5mm_P1.75mm, symbol LED:SK6812MINI

Commit message: Add files via upload
Parts:
- OL1: footprint oled:SSD1306-0.91-OLED-4pin-128x32 -> dp1:SSD1306-0.91-OLED-4pin-128x32
Connections:
- net GND: now also OL1.1 (GND); no longer OL1.4 (GND)
- net at U1.12 (3V3): now also OL1.2 (VCC); no longer OL1.3 (VCC)
- net at U1.5 (GPIO6/SDA): now also OL1.4 (SDA); no longer OL1.1 (SDA)
- net at U1.6 (GPIO7/SCL): now also OL1.3 (SCL); no longer OL1.2 (SCL)
