File: PCB/usbcmacropad.kicad_pcb (KiCad board)
At the start: 2 copper layers, 81 x 42.9 mm, 7 parts, among them SW1 SW_Push, SW2 SW_Push, SW3 SW_Push, SW4 SW_Push, U1 XIAO-RP2040-DIP

Commit message: Add files via upload
Parts:
- removed D1: SK6812MINI, LED_SMD:LED_SK6812MINI_PLCC4_3.5x3.5mm_P1.75mm
Routing:
- net +5V: track 14.5 -> 0.00 mm
- net Net-(OL1-SDA): track 60.5 -> 54.1 mm
- net GND: track 178.5 -> 176.7 mm

Commit message: Add files via upload
Parts:
- OL1: footprint oled:SSD1306-0.91-OLED-4pin-128x32 -> dp1:SSD1306-0.91-OLED-4pin-128x32
- moved OL1 40.6 mm to (107.0, 78.0), turned to 0 degrees
Connections:
- OL1 pad 1: Net-(OL1-SDA) -> GND
- OL1 pad 2: Net-(OL1-SCL) -> Net-(OL1-VCC)
- OL1 pad 3: Net-(OL1-VCC) -> Net-(OL1-SCL)
- OL1 pad 4: GND -> Net-(OL1-SDA)
Routing:
- net GND: track 176.7 -> 211.0 mm
- net Net-(OL1-VCC): track 22.8 -> 57.1 mm
- net Net-(OL1-SCL): track 40.1 -> 74.4 mm
- net Net-(OL1-SDA): track 54.1 -> 86.5 mm
